File: kicad/freepdk.sch (KiCad schematic (older format))
At the start: 56 parts, among them J1 MiniUSB, J2 SWD, J3 Conn_01x08, J4 Conn_01x08, J5 Conn_01x02, U1 STM32F072C8Tx, U2 XC6206P332MR, U3 MT3608, U4 LM2904DR2G, Y1 8MHz

Commit message: Second revision - Added fuse, improved routing, changed pcb dimentsions
Parts:
- added F1: PTC 0.5A 6V, Fuse:Fuse_0805_2012Metric_Pad1.15x1.40mm_HandSolder, symbol Device:Polyfuse
Connections:
- net +5V: now also F1.1; no longer J1.1 (VBUS)
- new net: F1.2, J1.1 (VBUS)
Changed lines of the file:
@@
 encoding utf-8
 Sheet 1 1
-Title "easypdkprog-lite-handsolder"
+Title "easy-pdk-mini"
 Date "2020-09-06"
 Rev "2"
@@
 Comment2 "Original hardware: https://github.com/free-pdk/easy-pdk-programmer-hardware"
 Comment3 "Based on easypdkprog-lite version of tim_ EEVBlog user"
-Comment4 ""
+Comment4 "https://github.com/pacmancoder/easy-pdk-mini"
 $EndDescr
 $Comp
@@
 Wire Wire Line
 	5100 7150 5100 7200
-Wire Wire Line
-	5500 6550 5600 6550
 $Comp
 L power:+5V #PWR0123
 U 1 1 5F570F25
-P 5600 6250
-F 0 "#PWR0123" H 5600 6100 50  0001 C CNN
-F 1 "+5V" H 5615 6423 50  0000 C CNN
-F 2 "" H 5600 6250 50  0001 C CNN
-F 3 "" H 5600 6250 50  0001 C CNN
-	1    5600 6250
+P 6600 6350
+F 0 "#PWR0123" H 6600 6200 50  0001 C CNN
+F 1 "+5V" H 6615 6523 50  0000 C CNN
+F 2 "" H 6600 6350 50  0001 C CNN
+F 3 "" H 6600 6350 50  0001 C CNN
+	1    6600 6350
 	1    0    0    -1
 $EndComp
@@
 Wire Wire Line
 	4200 1200 4200 1250
-Wire Wire Line
-	5600 6250 5600 6550
 Wire Wire Line
 	6600 1150 6600 1300
@@
 Wire Wire Line
 	5200 4650 5200 4800
+$Comp
+L Device:Polyfuse F1
+U 1 1 5F5CC5BA
+P 5950 6550
+F 0 "F1" V 5725 6550 50  0000 C CNN
+F 1 "PTC 0.5A 6V" V 5816 6550 50  0000 C CNN
+F 2 "Fuse:Fuse_0805_2012Metric_Pad1.15x1.40mm_HandSolder" H 6000 6350 50  0001 L CNN
+F 3 "~" H 5950 6550 50  0001 C CNN
+	1    5950 6550
+	0    1    1    0
+$EndComp
+Wire Wire Line
+	5500 6550 5800 6550
+Wire Wire Line
+	6100 6550 6600 6550
+Wire Wire Line
+	6600 6550 6600 6350
 $EndSCHEMATC

Commit message: Fixed silkscreen and markings
Parts:
- D2: value LED -> LED1
- D3: value LED -> LED2
- D4: value LED -> LED3
- J3: value Conn_01x08 -> CONN_L
- J4: value Conn_01x08 -> CONN_R
Changed lines of the file:
@@
 P 9050 3950
 F 0 "J3" H 9130 3942 50  0000 L CNN
-F 1 "Conn_01x08" H 9130 3851 50  0000 L CNN
+F 1 "CONN_L" H 9130 3851 50  0000 L CNN
 F 2 "Connector_PinSocket_2.54mm:PinSocket_1x08_P2.54mm_Vertical" H 9050 3950 50  0001 C CNN
 F 3 "~" H 9050 3950 50  0001 C CNN
@@
 P 10400 3950
 F 0 "J4" H 10480 3942 50  0000 L CNN
-F 1 "Conn_01x08" H 10480 3851 50  0000 L CNN
+F 1 "CONN_R" H 10480 3851 50  0000 L CNN
 F 2 "Connector_PinSocket_2.54mm:PinSocket_1x08_P2.54mm_Vertical" H 10400 3950 50  0001 C CNN
 F 3 "~" H 10400 3950 50  0001 C CNN
@@
 P 7600 2800
 F 0 "D2" V 7639 2683 50  0000 R CNN
-F 1 "LED" V 7548 2683 50  0000 R CNN
+F 1 "LED1" V 7548 2683 50  0000 R CNN
 F 2 "LED_SMD:LED_0805_2012Metric_Pad1.15x1.40mm_HandSolder" H 7600 2800 50  0001 C CNN
 F 3 "~" H 7600 2800 50  0001 C CNN
@@
 P 7950 2800
 F 0 "D3" V 7989 2683 50  0000 R CNN
-F 1 "LED" V 7898 2683 50  0000 R CNN
+F 1 "LED2" V 7898 2683 50  0000 R CNN
 F 2 "LED_SMD:LED_0805_2012Metric_Pad1.15x1.40mm_HandSolder" H 7950 2800 50  0001 C CNN
 F 3 "~" H 7950 2800 50  0001 C CNN
@@
 P 8300 2800
 F 0 "D4" V 8339 2683 50  0000 R CNN
-F 1 "LED" V 8248 2683 50  0000 R CNN
+F 1 "LED3" V 8248 2683 50  0000 R CNN
 F 2 "LED_SMD:LED_0805_2012Metric_Pad1.15x1.40mm_HandSolder" H 8300 2800 50  0001 C CNN
 F 3 "~" H 8300 2800 50  0001 C CNN

Commit message: Revision 3 - Applied suggestions from review, prepared gerbers
Parts:
- D2: value LED1 -> LED
- D3: value LED2 -> LED
- D4: value LED3 -> LED
Changed lines of the file:
@@
 Title "easy-pdk-mini"
 Date "2020-09-06"
-Rev "2"
+Rev "3"
 Comp "Vladislav Nikonov aka pacmancoder"
 Comment1 "pacmancoder.xyz"
@@
 P 7600 2800
 F 0 "D2" V 7639 2683 50  0000 R CNN
-F 1 "LED1" V 7548 2683 50  0000 R CNN
+F 1 "LED" V 7548 2683 50  0000 R CNN
 F 2 "LED_SMD:LED_0805_2012Metric_Pad1.15x1.40mm_HandSolder" H 7600 2800 50  0001 C CNN
 F 3 "~" H 7600 2800 50  0001 C CNN
@@
 P 7950 2800
 F 0 "D3" V 7989 2683 50  0000 R CNN
-F 1 "LED2" V 7898 2683 50  0000 R CNN
+F 1 "LED" V 7898 2683 50  0000 R CNN
 F 2 "LED_SMD:LED_0805_2012Metric_Pad1.15x1.40mm_HandSolder" H 7950 2800 50  0001 C CNN
 F 3 "~" H 7950 2800 50  0001 C CNN
@@
 P 8300 2800
 F 0 "D4" V 8339 2683 50  0000 R CNN
-F 1 "LED3" V 8248 2683 50  0000 R CNN
+F 1 "LED" V 8248 2683 50  0000 R CNN
 F 2 "LED_SMD:LED_0805_2012Metric_Pad1.15x1.40mm_HandSolder" H 8300 2800 50  0001 C CNN
 F 3 "~" H 8300 2800 50  0001 C CNN

Commit message: Revision 3 patch: Replaced wrong opamp; Removed logo from BOM
Parts:
- U4: value LM2904DR2G -> LM358DR2G
Changed lines of the file:
@@
 Title "easy-pdk-mini"
 Date "2020-09-06"
-Rev "3"
+Rev "4"
 Comp "Vladislav Nikonov aka pacmancoder"
 Comment1 "pacmancoder.xyz"
@@
 P 3500 3900
 F 0 "U4" H 3750 4200 50  0000 C CNN
-F 1 "LM2904DR2G" H 3800 4100 50  0000 C CNN
+F 1 "LM358DR2G" H 3800 4100 50  0000 C CNN
 F 2 "Package_SO:SOIC-8_3.9x4.9mm_P1.27mm" H 3500 3900 50  0001 C CNN
 F 3 "http://www.ti.com/lit/ds/symlink/lm2904-n.pdf" H 3500 3900 50  0001 C CNN
@@
 P 3450 5150
 F 0 "U4" H 3700 5450 50  0000 C CNN
-F 1 "LM2904DR2G" H 3750 5350 50  0000 C CNN
+F 1 "LM358DR2G" H 3750 5350 50  0000 C CNN
 F 2 "Package_SO:SOIC-8_3.9x4.9mm_P1.27mm" H 3450 5150 50  0001 C CNN
 F 3 "http://www.ti.com/lit/ds/symlink/lm2904-n.pdf" H 3450 5150 50  0001 C CNN
@@
 P 3500 6150
 F 0 "U4" V 3175 6150 50  0000 C CNN
-F 1 "LM2904DR2G" V 3250 6150 50  0000 C CNN
+F 1 "LM358DR2G" V 3250 6150 50  0000 C CNN
 F 2 "Package_SO:SOIC-8_3.9x4.9mm_P1.27mm" H 3500 6150 50  0001 C CNN
 F 3 "http://www.ti.com/lit/ds/symlink/lm2904-n.pdf" H 3500 6150 50  0001 C CNN

Commit message: Fixed issue with wrong opamp wiring
Connections:
- net DAC_VDD: now also U4.3 (+); no longer U4.2 (-)
- net DAC_VPP: now also U4.5 (+); no longer U4.6 (-)
- net at R11.1, R12.2: now also U4.2 (-); no longer U4.3 (+)
- net at R14.1, R15.2: now also U4.6 (-); no longer U4.5 (+)
Changed lines of the file:
@@
 Sheet 1 1
 Title "easy-pdk-mini"
-Date "2020-09-06"
-Rev "4"
+Date "2020-09-19"
+Rev "5"
 Comp "Vladislav Nikonov aka pacmancoder"
 Comment1 "pacmancoder.xyz"
@@
 U 1 1 5F7D7408
 P 3500 3900
-F 0 "U4" H 3750 4200 50  0000 C CNN
-F 1 "LM358DR2G" H 3800 4100 50  0000 C CNN
+F 0 "U4" H 3750 3550 50  0000 C CNN
+F 1 "LM358DR2G" H 3600 3450 50  0000 C CNN
 F 2 "Package_SO:SOIC-8_3.9x4.9mm_P1.27mm" H 3500 3900 50  0001 C CNN
 F 3 "http://www.ti.com/lit/ds/symlink/lm2904-n.pdf" H 3500 3900 50  0001 C CNN
 	1    3500 3900
-	1    0    0    -1
+	1    0    0    1
 $EndComp
 $Comp
@@
 U 2 1 5F7D92C5
 P 3450 5150
-F 0 "U4" H 3700 5450 50  0000 C CNN
-F 1 "LM358DR2G" H 3750 5350 50  0000 C CNN
+F 0 "U4" H 3700 4800 50  0000 C CNN
+F 1 "LM358DR2G" H 3550 4700 50  0000 C CNN
 F 2 "Package_SO:SOIC-8_3.9x4.9mm_P1.27mm" H 3450 5150 50  0001 C CNN
 F 3 "http://www.ti.com/lit/ds/symlink/lm2904-n.pdf" H 3450 5150 50  0001 C CNN
 	2    3450 5150
-	1    0    0    -1
-$EndComp
-$Comp
+	1    0    0    1
+$EndComp
+$Comp

Commit message: Updated PCB to use USB-B port instead of Mini-usb
Parts:
- removed J1: MiniUSB, Connector_USB:USB_Mini-B_Lumberg_2486_01_Horizontal, symbol Connector:USB_B_Mini
- added J1: USB_B, Connector_USB:USB_B_OST_USB-B1HSxx_Horizontal, symbol Connector:USB_B
Connections:
- net GND: now also J1.4 (GND), J1.5 (Shield)
- net USB_D+: now also J1.3 (D+)
- net USB_D-: now also J1.2 (D-)
- net at F1.2: now also J1.1 (VBUS)
- no-connect marks 27 -> 26
Changed lines of the file:
@@
 Sheet 1 1
 Title "easy-pdk-mini"
-Date "2020-09-19"
-Rev "5"
+Date "2020-09-23"
+Rev "1.1.0"
 Comp "Vladislav Nikonov aka pacmancoder"
 Comment1 "pacmancoder.xyz"
@@
 Wire Wire Line
 	7950 2050 7950 2150
-$Comp
-L Device:Crystal Y1
-U 1 1 5F1F422C
-P 9200 2700
-F 0 "Y1" H 9200 2432 50  0000 C CNN
-F 1 "8MHz" H 9200 2523 50  0000 C CNN
-F 2 "Crystal:Crystal_SMD_HC49-SD" H 9200 2700 50  0001 C CNN
-F 3 "~" H 9200 2700 50  0001 C CNN
-	1    9200 2700
-	-1   0    0    1
-$EndComp
 $Comp
 L Device:C C9
@@
 Wire Wire Line
 	1350 2100 1350 1750
-NoConn ~ 5500 6950
 Wire Wire Line
 	5200 7200 5200 7150
@@
 F 3 "" H 5200 7250 50  0001 C CNN
 	1    5200 7250
-	1    0    0    -1
-$EndComp
-$Comp
-L Connector:USB_B_Mini J1
-U 1 1 5F56BF1B
-P 5200 6750
-F 0 "J1" H 5257 7217 50  0000 C CNN
-F 1 "MiniUSB" H 5257 7126 50  0000 C CNN
-F 2 "Connector_USB:USB_Mini-B_Lumberg_2486_01_Horizontal" H 5350 6700 50  0001 C CNN
-F 3 "~" H 5350 6700 50  0001 C CNN
-	1    5200 6750
 	1    0    0    -1
 $EndComp
@@
 Wire Wire Line
 	6600 6550 6600 6350
+$Comp
+L Connector:USB_B J1
+U 1 1 5F6E3453
+P 5200 6750
+F 0 "J1" H 5257 7217 50  0000 C CNN
+F 1 "USB_B" H 5257 7126 50  0000 C CNN
+F 2 "Connector_USB:USB_B_OST_USB-B1HSxx_Horizontal" H 5350 6700 50  0001 C CNN
+F 3 " ~" H 5350 6700 50  0001 C CNN
+	1    5200 6750
+	1    0    0    -1
+$EndComp
+$Comp
+L Device:Crystal Y1
+U 1 1 5F1F422C
+P 9200 2700
+F 0 "Y1" H 9200 2432 50  0000 C CNN
+F 1 "8MHz" H 9200 2523 50  0000 C CNN
+F 2 "Crystal:Crystal_SMD_HC49-SD" H 9200 2700 50  0001 C CNN
+F 3 "~" H 9200 2700 50  0001 C CNN
+	1    9200 2700
+	-1   0    0    1
+$EndComp
 $EndSCHEMATC
